File: Schematics/KiCad/Jettabrain/Jettabrain.kicad_sch (KiCad schematic)
At the start: 12 parts, among them J1 Conn_01x07_Pin, J2 Conn_01x07_Pin, J3 Conn_01x04, J4 Conn_01x07_Pin, J5 Conn_01x14_Pin, J6 Conn_01x08_Pin, J7 Conn_01x01_Pin

Commit message: Generated Gerber Files
Parts:
- renumbered J1 to +5V1, A1 to Arduino_Nano1, J3 to Display1, J4 to GND1, J2 to I/O1
Changed lines of the file:
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@@
     (pin "12")
     (instances
-      (project "KCT"
+      (project "Jettabrain"
         (path "/008ca40f-114f-48cb-bea6-2f15c29a817d"
           (reference "J5") (unit 1)
@@
     (pin "1")
     (instances
-      (project "KCT"
+      (project "Jettabrain"
         (path "/008ca40f-114f-48cb-bea6-2f15c29a817d"
           (reference "J7") (unit 1)
@@
   (symbol (lib_id "Connector:Conn_01x07_Pin") (at 110.49 124.46 90) (unit 1)
     (in_bom yes) (on_board yes) (dnp no)
-    (property "Reference" "J2" (at 110.49 129.54 90)
+    (property "Reference" "I/O1" (at 110.49 129.54 90)
       (effects (font (size 1.27 1.27)))
     )
@@
     (pin "2")
     (instances
-      (project "KCT"
-        (path "/008ca40f-114f-48cb-bea6-2f15c29a817d"
-          (reference "J2") (unit 1)
+      (project "Jettabrain"
+        (path "/008ca40f-114f-48cb-bea6-2f15c29a817d"
+          (reference "I/O1") (unit 1)
         )
       )
@@
   (symbol (lib_id "Connector:Conn_01x07_Pin") (at 187.96 135.89 90) (unit 1)
     (in_bom yes) (on_board yes) (dnp no) (fields_autoplaced)
-    (property "Reference" "J4" (at 187.96 138.43 90)
+    (property "Reference" "GND1" (at 187.96 138.43 90)
       (effects (font (size 1.27 1.27)))
     )
@@
     (pin "2")
     (instances
-      (project "KCT"
-        (path "/008ca40f-114f-48cb-bea6-2f15c29a817d"
-          (reference "J4") (unit 1)
+      (project "Jettabrain"
+        (path "/008ca40f-114f-48cb-bea6-2f15c29a817d"
+          (reference "GND1") (unit 1)
         )
       )
@@
     (pin "2")
     (instances
-      (project "KCT"
+      (project "Jettabrain"
         (path "/008ca40f-114f-48cb-bea6-2f15c29a817d"
           (reference "R1") (unit 1)
@@
   (symbol (lib_id "Connector:Conn_01x07_Pin") (at 185.42 66.04 270) (unit 1)
     (in_bom yes) (on_board yes) (dnp no) (fields_autoplaced)
-    (property "Reference" "J1" (at 185.42 60.96 90)
+    (property "Reference" "+5V1" (at 185.42 60.96 90)
       (effects (font (size 1.27 1.27)))
     )
@@
     (pin "2")
     (instances
-      (project "KCT"
-        (path "/008ca40f-114f-48cb-bea6-2f15c29a817d"
-          (reference "J1") (unit 1)
+      (project "Jettabrain"
+        (path "/008ca40f-114f-48cb-bea6-2f15c29a817d"
+          (reference "+5V1") (unit 1)
         )
       )
@@
     (pin "1")
     (instances
-      (project "KCT"
+      (project "Jettabrain"
         (path "/008ca40f-114f-48cb-bea6-2f15c29a817d"
           (reference "#PWR01") (unit 1)
@@
     (pin "2")
     (instances
-      (project "KCT"
+      (project "Jettabrain"
         (path "/008ca40f-114f-48cb-bea6-2f15c29a817d"
           (reference "R3") (unit 1)
@@
     (pin "2")
     (instances
-      (project "KCT"
+      (project "Jettabrain"
         (path "/008ca40f-114f-48cb-bea6-2f15c29a817d"
           (reference "R2") (unit 1)
@@
     (pin "3")
     (instances
-      (project "KCT"
+      (project "Jettabrain"
         (path "/008ca40f-114f-48cb-bea6-2f15c29a817d"
           (reference "J6") (unit 1)
@@
     (pin "2")
     (instances
-      (project "KCT"
+      (project "Jettabrain"
         (path "/008ca40f-114f-48cb-bea6-2f15c29a817d"
           (reference "R4") (unit 1)
@@
     (pin "1")
     (instances
-      (project "KCT"
+      (project "Jettabrain"
         (path "/008ca40f-114f-48cb-bea6-2f15c29a817d"
           (reference "#PWR02") (unit 1)
@@
   (symbol (lib_id "Connector:Conn_01x04_Pin") (at 191.77 111.76 180) (unit 1)
     (in_bom yes) (on_board yes) (dnp no)
-    (property "Reference" "J3" (at 189.23 118.11 0)
+    (property "Reference" "Display1" (at 189.23 118.11 0)
       (effects (font (size 1.27 1.27)))
     )
@@
     (pin "4")
     (instances
-      (project "KCT"
-        (path "/008ca40f-114f-48cb-bea6-2f15c29a817d"
-          (reference "J3") (unit 1)
+      (project "Jettabrain"
+        (path "/008ca40f-114f-48cb-bea6-2f15c29a817d"
+          (reference "Display1") (unit 1)
         )
       )
@@
   (symbol (lib_id "MCU_Module:Arduino_Nano_v3.x") (at 152.4 101.6 0) (unit 1)
     (in_bom yes) (on_board yes) (dnp no) (fields_autoplaced)
-    (property "Reference" "A1" (at 157.1341 127 0)
+    (property "Reference" "Arduino_Nano1" (at 157.1341 127 0)
       (effects (font (size 1.27 1.27)) (justify left) hide)
     )
@@
     (pin "23")
     (instances
-      (project "KCT"
-        (path "/008ca40f-114f-48cb-bea6-2f15c29a817d"
-          (reference "A1") (unit 1)
-        )
-      )
+      (project "Jettabrain"
+        (path "/008ca40f-114f-48cb-bea6-2f15c29a817d"
+          (reference "Arduino_Nano1") (unit 1)
+        )
+      )
