File: Schematics/KiCad/Jettabrain/Jettabrain.kicad_pcb (KiCad board)
At the start: 2 copper layers, 38.1 x 50.8 mm, 12 parts, among them J1 Conn_01x07, J2 Conn_01x07_Pin, J3 Conn_01x04, J4 Conn_01x07, J5 Conn_01x14_Pin, J6 Conn_01x08_Pin, J7 Conn_01x01

Commit message: Generated Gerber Files
Parts:
- +5V1: renamed from J1; value Conn_01x07 -> Conn_01x07_Pin
- GND1: renamed from J4; value Conn_01x07 -> Conn_01x07_Pin
- J7: value Conn_01x01 -> Conn_01x01_Pin
- renumbered A1 to Arduino_Nano1, J3 to Display1, J2 to I/O1
Routing:
- net Net-(Arduino_Nano1-D6): track 19.0 -> 20.2 mm
- net Net-(Arduino_Nano1-D9): track 38.8 -> 39.8 mm
- net Net-(Arduino_Nano1-D5): track 17.7 -> 18.7 mm
- net Net-(Arduino_Nano1-D3): track 28.0 -> 29.0 mm
- net Net-(Arduino_Nano1-D2): track 36.4 -> 37.4 mm
- net Net-(Arduino_Nano1-D1/TX): track 6.88 -> 7.89 mm
- net Net-(Arduino_Nano1-D0/RX): track 7.51 -> 8.53 mm
- net Net-(Arduino_Nano1-D8): track 21.2 -> 22.2 mm
- net Net-(Arduino_Nano1-D7): track 19.9 -> 21.0 mm
- net Net-(Arduino_Nano1-D4): track 16.0 -> 16.9 mm
- net Net-(Arduino_Nano1-GND-Pad4): track 38.4 -> 37.6 mm
Other:
- board text added: "JLCJLCJLCJLC"

Commit message: PCB Updates
Parts:
- added +12V1: Conn_01x01_Pin, Connector_PinHeader_2.54mm:PinHeader_1x01_P2.54mm_Horizontal, F.Cu at (129.5, 86.6)
- +5V1, GND1, I/O1: footprint Connector_PinHeader_1.00mm:PinHeader_1x07_P1.00mm_Horizontal -> Connector_PinHeader_2.54mm:PinHeader_1x07_P2.54mm_Horizontal
- Display1: footprint Connector_PinHeader_1.00mm:PinHeader_1x04_P1.00mm_Horizontal -> Connector_PinHeader_2.54mm:PinHeader_1x04_P2.54mm_Horizontal
- J5: footprint Connector_PinHeader_1.00mm:PinHeader_1x14_P1.00mm_Vertical -> Connector_PinHeader_2.54mm:PinHeader_1x14_P2.54mm_Vertical; moved to B.Cu
- J6: footprint Connector_PinHeader_1.00mm:PinHeader_1x08_P1.00mm_Vertical -> Connector_PinHeader_2.54mm:PinHeader_1x08_P2.54mm_Horizontal
- J7: footprint Connector_PinHeader_1.00mm:PinHeader_1x01_P1.00mm_Vertical -> Connector_PinHeader_2.54mm:PinHeader_1x01_P2.54mm_Horizontal
- R1, R2, R3, R4: moved to B.Cu
- moved R1 17.5 mm to (142.0, 105.7), turned to 180 degrees
- moved R2 17.5 mm to (142.0, 109.0), turned to 180 degrees
- moved R3 17.5 mm to (142.0, 112.3), turned to 180 degrees
- moved R4 17.5 mm to (142.0, 115.5), turned to 180 degrees
- moved J6 10.9 mm to (155.3, 98.6)
- moved GND1 9.94 mm to (124.2, 81.8)
- moved J5 6.39 mm to (130.6, 93.5), turned to 180 degrees
- moved J7 2.61 mm to (155.3, 120.7)
- moved Display1 2.46 mm to (156.3, 86.9)
- moved I/O1 1.67 mm to (126.0, 110.2)
- moved +5V1 0.45 mm to (143.5, 81.8)
Connections:
- Arduino_Nano1 pad 30: +12V -> Net-(+12V1-Pin_1)
- I/O1 pad 1: Net-(Arduino_Nano1-D9) -> Net-(Arduino_Nano1-D13)
- I/O1 pad 2: Net-(Arduino_Nano1-D10) -> Net-(Arduino_Nano1-D12)
- I/O1 pad 3: Net-(Arduino_Nano1-D13) -> Net-(Arduino_Nano1-D10)
- I/O1 pad 4: Net-(Arduino_Nano1-D12) -> Net-(Arduino_Nano1-D9)
- R1 pad 2: Net-(Arduino_Nano1-D9) -> Net-(Arduino_Nano1-D13)
- R2 pad 2: Net-(Arduino_Nano1-D10) -> Net-(Arduino_Nano1-D12)
- R3 pad 2: Net-(Arduino_Nano1-D13) -> Net-(Arduino_Nano1-D10)
- R4 pad 2: Net-(Arduino_Nano1-D12) -> Net-(Arduino_Nano1-D9)
Routing:
- net Net-(Arduino_Nano1-D2): track 37.4 -> 9.27 mm
- net Net-(Arduino_Nano1-D10): track 54.0 -> 32.1 mm, vias 3 -> 1
- net Net-(+12V1-Pin_1): track 0.00 -> 21.1 mm
- net Net-(Arduino_Nano1-D3): track 29.0 -> 10.1 mm, vias 1 -> 0
- net Net-(Arduino_Nano1-D8): track 22.2 -> 4.06 mm
- net Net-(Arduino_Nano1-D7): track 21.0 -> 4.06 mm
- net Net-(Arduino_Nano1-D6): track 20.2 -> 4.06 mm
- net Net-(Arduino_Nano1-D5): track 18.7 -> 4.06 mm
- net Net-(Arduino_Nano1-GND-Pad4): track 37.6 -> 23.2 mm, vias 1 -> 0
- net Net-(Arduino_Nano1-A7): track 18.6 -> 5.46 mm
- net Net-(Arduino_Nano1-D4): track 16.9 -> 4.06 mm
- net Net-(Arduino_Nano1-D9): track 39.8 -> 27.4 mm, vias 1 -> 0
- net Net-(Arduino_Nano1-D13): track 55.5 -> 67.2 mm
- net Net-(Arduino_Nano1-A6): track 17.1 -> 5.46 mm
- net Net-(Arduino_Nano1-A5): track 30.1 -> 21.0 mm, vias 1 -> 0
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