File: Schematics/KiCad/Jettabrain_OLD/Jettabrain_OLD.kicad_sch (KiCad schematic)
At the start: 13 parts, among them J5 Conn_01x14_Pin, J6 Conn_01x08_Pin, J7 Conn_01x01_Pin

Commit message: PCB Updates
Parts:
- removed +12V1: Conn_01x01_Pin, Connector_PinHeader_2.54mm:PinHeader_1x01_P2.54mm_Horizontal, symbol Connector:Conn_01x01_Pin
- +5V1, GND1, I/O1: footprint Connector_PinHeader_2.54mm:PinHeader_1x07_P2.54mm_Horizontal -> Connector_PinHeader_1.00mm:PinHeader_1x07_P1.00mm_Horizontal
- Display1: footprint Connector_PinHeader_2.54mm:PinHeader_1x04_P2.54mm_Horizontal -> Connector_PinHeader_1.00mm:PinHeader_1x04_P1.00mm_Horizontal
- J5: footprint Connector_PinHeader_2.54mm:PinHeader_1x14_P2.54mm_Vertical -> Connector_PinHeader_1.00mm:PinHeader_1x14_P1.00mm_Vertical
- J6: footprint Connector_PinHeader_2.54mm:PinHeader_1x08_P2.54mm_Horizontal -> Connector_PinHeader_1.00mm:PinHeader_1x08_P1.00mm_Vertical
- J7: footprint Connector_PinHeader_2.54mm:PinHeader_1x01_P2.54mm_Horizontal -> Connector_PinHeader_1.00mm:PinHeader_1x01_P1.00mm_Vertical
Connections:
- net at Arduino_Nano1.12 (D9), J5.10 (Pin_10): now also I/O1.1 (Pin_1), R1.2; no longer I/O1.4 (Pin_4), R4.2
- net at Arduino_Nano1.13 (D10), J5.11 (Pin_11): now also I/O1.2 (Pin_2), R2.2; no longer I/O1.3 (Pin_3), R3.2
- net at Arduino_Nano1.15 (D12), J5.13 (Pin_13): now also I/O1.4 (Pin_4), R4.2; no longer I/O1.2 (Pin_2), R2.2
- net at Arduino_Nano1.16 (D13), J5.14 (Pin_14): now also I/O1.3 (Pin_3), R3.2; no longer I/O1.1 (Pin_1), R1.2
- net +12V: now reaches Arduino_Nano1.30 (VIN)
Changed lines of the file:
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@@
   (junction (at 170.18 114.3) (diameter 0) (color 0 0 0 0)
   )
-  (junction (at 105.41 116.84) (diameter 0) (color 0 0 0 0)
-  )
   (junction (at 193.04 130.81) (diameter 0) (color 0 0 0 0)
   )
   (junction (at 154.94 128.27) (diameter 0) (color 0 0 0 0)
   )
-  (junction (at 110.49 111.76) (diameter 0) (color 0 0 0 0)
-  )
   (junction (at 185.42 71.12) (diameter 0) (color 0 0 0 0)
   )
+  (junction (at 110.49 116.84) (diameter 0) (color 0 0 0 0)
+  )
   (junction (at 190.5 71.12) (diameter 0) (color 0 0 0 0)
   )
@@
   (junction (at 107.95 102.87) (diameter 0) (color 0 0 0 0)
   )
-  (junction (at 107.95 113.03) (diameter 0) (color 0 0 0 0)
+  (junction (at 134.62 116.84) (diameter 0) (color 0 0 0 0)
   )
   (junction (at 182.88 130.81) (diameter 0) (color 0 0 0 0)
   )
-  (junction (at 102.87 118.11) (diameter 0) (color 0 0 0 0)
+  (junction (at 102.87 111.76) (diameter 0) (color 0 0 0 0)
   )
   (junction (at 139.7 119.38) (diameter 0) (color 0 0 0 0)
   )
+  (junction (at 105.41 113.03) (diameter 0) (color 0 0 0 0)
+  )
   (junction (at 138.43 111.76) (diameter 0) (color 0 0 0 0)
   )
@@
   (junction (at 105.41 102.87) (diameter 0) (color 0 0 0 0)
   )
-  (junction (at 134.62 116.84) (diameter 0) (color 0 0 0 0)
+  (junction (at 107.95 118.11) (diameter 0) (color 0 0 0 0)
   )
   (junction (at 170.18 111.76) (diameter 0) (color 0 0 0 0)
@@
     (stroke (width 0) (type default))
   )
+  (wire (pts (xy 105.41 113.03) (xy 138.43 113.03))
+    (stroke (width 0) (type default))
+  )
   (wire (pts (xy 170.18 114.3) (xy 182.88 114.3))
     (stroke (width 0) (type default))
@@
     (stroke (width 0) (type default))
   )
+  (wire (pts (xy 102.87 111.76) (xy 102.87 119.38))
+    (stroke (width 0) (type default))
+  )
   (wire (pts (xy 186.69 109.22) (xy 185.42 109.22))
     (stroke (width 0) (type default))
@@
     (stroke (width 0) (type default))
   )
-  (wire (pts (xy 102.87 118.11) (xy 139.7 118.11))
+  (wire (pts (xy 107.95 118.11) (xy 139.7 118.11))
     (stroke (width 0) (type default))
   )
@@
     (stroke (width 0) (type default))
   )
-  (wire (pts (xy 110.49 111.76) (xy 121.92 111.76))
-    (stroke (width 0) (type default))
-  )
   (wire (pts (xy 165.1 104.14) (xy 170.18 104.14))
     (stroke (width 0) (type default))
@@
     (stroke (width 0) (type default))
   )
-  (wire (pts (xy 107.95 113.03) (xy 138.43 113.03))
-    (stroke (width 0) (type default))
-  )
   (wire (pts (xy 115.57 93.98) (xy 115.57 119.38))
     (stroke (width 0) (type default))
   )
+  (wire (pts (xy 110.49 116.84) (xy 134.62 116.84))
+    (stroke (width 0) (type default))
+  )
   (wire (pts (xy 182.88 130.81) (xy 185.42 130.81))
     (stroke (width 0) (type default))
@@
     (stroke (width 0) (type default))
   )
-  (wire (pts (xy 102.87 110.49) (xy 102.87 118.11))
+  (wire (pts (xy 102.87 110.49) (xy 102.87 111.76))
     (stroke (width 0) (type default))
   )
@@
     (stroke (width 0) (type default))
   )
-  (wire (pts (xy 105.41 110.49) (xy 105.41 116.84))
+  (wire (pts (xy 105.41 110.49) (xy 105.41 113.03))
     (stroke (width 0) (type default))
   )
@@
     (stroke (width 0) (type default))
   )
+  (wire (pts (xy 102.87 111.76) (xy 121.92 111.76))
+    (stroke (width 0) (type default))
+  )
   (wire (pts (xy 182.88 113.03) (xy 186.69 113.03))
     (stroke (width 0) (type default))
@@
     (stroke (width 0) (type default))
   )
+  (wire (pts (xy 110.49 110.49) (xy 110.49 116.84))
+    (stroke (width 0) (type default))
+  )
   (wire (pts (xy 165.1 114.3) (xy 170.18 114.3))
     (stroke (width 0) (type default))
@@
     (stroke (width 0) (type default))
   )
-  (wire (pts (xy 110.49 111.76) (xy 110.49 119.38))
-    (stroke (width 0) (type default))
-  )
   (wire (pts (xy 165.1 119.38) (xy 170.18 119.38))
     (stroke (width 0) (type default))
   )
-  (wire (pts (xy 110.49 110.49) (xy 110.49 111.76))
+  (wire (pts (xy 110.49 116.84) (xy 110.49 119.38))
     (stroke (width 0) (type default))
   )
@@
     (stroke (width 0) (type default))
   )
-  (wire (pts (xy 107.95 113.03) (xy 107.95 119.38))
-    (stroke (width 0) (type default))
-  )
-  (wire (pts (xy 105.41 116.84) (xy 105.41 119.38))
-    (stroke (width 0) (type default))
-  )
   (wire (pts (xy 134.62 93.98) (xy 139.7 93.98))
     (stroke (width 0) (type default))
   )
+  (wire (pts (xy 149.86 73.66) (xy 149.86 76.2))
+    (stroke (width 0) (type default))
+  )
   (wire (pts (xy 138.43 110.49) (xy 138.43 109.22))
     (stroke (width 0) (type default))
@@
     (stroke (width 0) (type default))
   )
-  (wire (pts (xy 105.41 116.84) (xy 134.62 116.84))
-    (stroke (width 0) (type default))
-  )
-  (wire (pts (xy 102.87 118.11) (xy 102.87 119.38))
-    (stroke (width 0) (type default))
-  )
-  (wire (pts (xy 107.95 110.49) (xy 107.95 113.03))
-    (stroke (width 0) (type default))
-  )
-  (wire (pts (xy 149.86 73.66) (xy 149.86 76.2))
+  (wire (pts (xy 107.95 110.49) (xy 107.95 118.11))
     (stroke (width 0) (type default))
   )
@@
     (stroke (width 0) (type default))
   )
+  (wire (pts (xy 107.95 118.11) (xy 107.95 119.38))
+    (stroke (width 0) (type default))
+  )
+  (wire (pts (xy 105.41 113.03) (xy 105.41 119.38))
+    (stroke (width 0) (type default))
+  )
   (wire (pts (xy 170.18 111.76) (xy 184.15 111.76))
     (stroke (width 0) (type default))
   )
   (symbol (lib_id "Connector:Conn_01x14_Pin") (at 129.54 101.6 0) (unit 1)
-    (in_bom yes) (on_board yes) (dnp no)
+    (in_bom yes) (on_board yes) (dnp no) (fields_autoplaced)
     (property "Reference" "J5" (at 130.175 81.28 0)
       (effects (font (size 1.27 1.27)))
@@
       (effects (font (size 1.27 1.27)))
     )
-    (property "Footprint" "Connector_PinHeader_2.54mm:PinHeader_1x14_P2.54mm_Vertical" (at 129.54 101.6 0)
+    (property "Footprint" "Connector_PinHeader_1.00mm:PinHeader_1x14_P1.00mm_Vertical" (at 129.54 101.6 0)
       (effects (font (size 1.27 1.27)) hide)
     )
@@
       (effects (font (size 1.27 1.27)))
     )
-    (property "Footprint" "Connector_PinHeader_2.54mm:PinHeader_1x01_P2.54mm_Horizontal" (at 175.26 96.52 0)
+    (property "Footprint" "Connector_PinHeader_1.00mm:PinHeader_1x01_P1.00mm_Vertical" (at 175.26 96.52 0)
       (effects (font (size 1.27 1.27)) hide)
     )
@@
       (effects (font (size 1.27 1.27)))
     )
-    (property "Footprint" "Connector_PinHeader_2.54mm:PinHeader_1x07_P2.54mm_Horizontal" (at 110.49 124.46 0)
+    (property "Footprint" "Connector_PinHeader_1.00mm:PinHeader_1x07_P1.00mm_Horizontal" (at 110.49 124.46 0)
       (effects (font (size 1.27 1.27)) hide)
     )
@@
       (effects (font (size 1.27 1.27)))
     )
-    (property "Footprint" "Connector_PinHeader_2.54mm:PinHeader_1x07_P2.54mm_Horizontal" (at 187.96 135.89 0)
+    (property "Footprint" "Connector_PinHeader_1.00mm:PinHeader_1x07_P1.00mm_Horizontal" (at 187.96 135.89 0)
       (effects (font (size 1.27 1.27)) hide)
     )
@@
       (effects (font (size 1.27 1.27)))
     )
-    (property "Footprint" "Connector_PinHeader_2.54mm:PinHeader_1x07_P2.54mm_Horizontal" (at 185.42 66.04 0)
+    (property "Footprint" "Connector_PinHeader_1.00mm:PinHeader_1x07_P1.00mm_Horizontal" (at 185.42 66.04 0)
       (effects (font (size 1.27 1.27)) hide)
     )
@@
     )
   )
-  (symbol (lib_id "Connector:Conn_01x01_Pin") (at 149.86 68.58 270) (unit 1)
-    (in_bom yes) (on_board yes) (dnp no) (fields_autoplaced)
-    (property "Reference" "+12V1" (at 151.13 67.945 90)
-      (effects (font (size 1.27 1.27)) (justify left))
-    )
-    (property "Value" "Conn_01x01_Pin" (at 151.13 70.485 90)
-      (effects (font (size 1.27 1.27)) (justify left))
-    )
-    (property "Footprint" "Connector_PinHeader_2.54mm:PinHeader_1x01_P2.54mm_Horizontal" (at 149.86 68.58 0)
-      (effects (font (size 1.27 1.27)) hide)
-    )
-    (property "Datasheet" "~" (at 149.86 68.58 0)
-      (effects (font (size 1.27 1.27)) hide)
-    )
-    (pin "1")
-    (instances
-      (project "Jettabrain"
-        (path "/008ca40f-114f-48cb-bea6-2f15c29a817d"
-          (reference "+12V1") (unit 1)
+  (symbol (lib_id "power:+12V") (at 149.86 73.66 0) (unit 1)
+    (in_bom yes) (on_board yes) (dnp no)
+    (property "Reference" "#PWR01" (at 149.86 77.47 0)
+      (effects (font (size 1.27 1.27)) hide)
+    )
+    (property "Value" "+12V" (at 149.86 69.85 0)
+      (effects (font (size 1.27 1.27)))
+    )
+    (property "Footprint" "" (at 149.86 73.66 0)
+      (effects (font (size 1.27 1.27)) hide)
+    )
+    (property "Datasheet" "" (at 149.86 73.66 0)
+      (effects (font (size 1.27 1.27)) hide)
+    )
+    (pin "1")
+    (instances
+      (project "Jettabrain"
+        (path "/008ca40f-114f-48cb-bea6-2f15c29a817d"
+          (reference "#PWR01") (unit 1)
         )
       )
@@
       (effects (font (size 1.27 1.27)) (justify right))
     )
-    (property "Footprint" "Connector_PinHeader_2.54mm:PinHeader_1x08_P2.54mm_Horizontal" (at 175.26 111.76 0)
+    (property "Footprint" "Connector_PinHeader_1.00mm:PinHeader_1x08_P1.00mm_Vertical" (at 175.26 111.76 0)
       (effects (font (size 1.27 1.27)) hide)
     )
@@
       (effects (font (size 1.27 1.27)))
     )
-    (property "Footprint" "Connector_PinHeader_2.54mm:PinHeader_1x04_P2.54mm_Horizontal" (at 191.77 111.76 0)
-      (effects (font (size 1.27 1.27)) hide)
-    )
+    (property "Footprint" "Connector_PinHeader_1.00mm:PinHeader_1x04_P1.00mm_Horizontal" (at 191.77 111.76 0)
+      (effects (font (size 1.27 1.27)) hide)
+    )
